File: Kicad/cage_LEDbutton_pi/cage_LEDbutton_pi.kicad_pcb (KiCad board)
At the start: 2 copper layers, 2.2 x 0.7 mm, 32 parts, among them J1 Raspberry_Pi_2_3, J2 USB_B_Micro, Q1 BSN20, Q2 BSN20, Q3 BSN20, Q4 BSN20, U1 LED_Button_connector, U2 LED_Button_connector, U3 LED_Button_connector, U4 LED_Button_connector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

Commit message: Updating the edges of the boards
Other:
- board size 2.2 x 0.7 mm -> 62.1 x 72.2 mm
Changed lines of the file:
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@@
-(kicad_pcb (version 20171130) (host pcbnew 5.1.4-e60b266~84~ubuntu18.04.1)
+(kicad_pcb (version 20171130) (host pcbnew 5.1.5-52549c5~84~ubuntu18.04.1)
   (general
     (thickness 1.6)
-    (drawings 5)
+    (drawings 6)
     (tracks 357)
     (zones 0)
@@
       (net 33 +5V))
   )
-  (gr_line (start 127 65.024) (end 127.254 65.024) (layer F.SilkS) (width 0.12))
-  (gr_line (start 127 136.906) (end 127 65.024) (layer F.SilkS) (width 0.12))
-  (gr_line (start 188.722 136.906) (end 127 136.906) (layer F.SilkS) (width 0.12))
-  (gr_line (start 188.722 65.024) (end 188.722 136.906) (layer F.SilkS) (width 0.12))
-  (gr_line (start 127.254 65.024) (end 188.722 65.024) (layer F.SilkS) (width 0.12))
+  (gr_line (start 126.6952 65.0113) (end 126.7968 65.0113) (layer Edge.Cuts) (width 0.05))
+  (gr_line (start 126.6952 65.0113) (end 126.7714 65.0113) (layer Edge.Cuts) (width 0.1))
+  (gr_line (start 126.6952 137.2108) (end 126.6952 65.0113) (layer Edge.Cuts) (width 0.1))
+  (gr_line (start 188.7728 137.2108) (end 126.6952 137.2108) (layer Edge.Cuts) (width 0.1))
+  (gr_line (start 188.7728 65.0113) (end 188.7728 137.2108) (layer Edge.Cuts) (width 0.1))
+  (gr_line (start 126.7841 65.0113) (end 188.7728 65.0113) (layer Edge.Cuts) (width 0.1))
   (segment (start 145.001 82.804) (end 147.916 85.719) (width 0.25) (layer F.Cu) (net 1))
   (segment (start 133.35 82.804) (end 145.001 82.804) (width 0.25) (layer F.Cu) (net 1))
