File: Kicad/cage_LEDbutton_pi/cage_LEDbutton_pi.sch (KiCad schematic (older format))
At the start: 32 parts, among them J1 Raspberry_Pi_2_3, J2 USB_B_Micro, Q1 BSN20, Q2 BSN20, Q3 BSN20, Q4 BSN20, U1 LED_Button_connector, U2 LED_Button_connector, U3 LED_Button_connector, U4 LED_Button_connector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

Commit message: Updating kicad libraries so prevent broken links
Parts:
- U1, U2, U3, U4, U5, U6, U7, U8: symbol MillerLab_CommonComponents:LED_Button_connector -> cage_LEDbutton_pi-rescue:LED_Button_connector-MillerLab_CommonComponents
- U9: symbol additional_LED_drivers:LED_shift_register_SPI -> cage_LEDbutton_pi-rescue:LED_shift_register_SPI-additional_LED_drivers
Changed lines of the file:
@@
 EESchema Schematic File Version 4
-LIBS:cage_LEDbutton_pi-cache
 EELAYER 30 0
 EELAYER END
@@
 $EndDescr
 $Comp
-L additional_LED_drivers:LED_shift_register_SPI U9
+L cage_LEDbutton_pi-rescue:LED_shift_register_SPI-additional_LED_drivers U9
 U 1 1 5DC3894E
 P 5550 4250
@@
 F 1 "LED_shift_register_SPI" H 5575 4274 50  0000 C CNN
 F 2 "Package_SO:HTSSOP-28-1EP_4.4x9.7mm_P0.65mm_EP3.4x9.5mm" H 5550 4250 50  0001 C CNN
-F 3 "/home/kevin/Documents/kicad/Libraries/PCA9745B.pdf" H 5550 4250 50  0001 C CNN
+F 3 "/home/kevin/Documents/git/proc-kevin/Kicad/Libraries/PCA9745B.pdf" H 5550 4250 50  0001 C CNN
 	1    5550 4250
 	-1   0    0    -1
@@
 	4900 4400 5050 4400
 $Comp
-L MillerLab_CommonComponents:LED_Button_connector U2
+L cage_LEDbutton_pi-rescue:LED_Button_connector-MillerLab_CommonComponents U2
 U 1 1 5DCB3B09
 P 1350 5850
@@
 $EndComp
 $Comp
-L MillerLab_CommonComponents:LED_Button_connector U3
+L cage_LEDbutton_pi-rescue:LED_Button_connector-MillerLab_CommonComponents U3
 U 1 1 5DCBFAD0
 P 1350 6500
@@
 $EndComp
 $Comp
-L MillerLab_CommonComponents:LED_Button_connector U4
+L cage_LEDbutton_pi-rescue:LED_Button_connector-MillerLab_CommonComponents U4
 U 1 1 5DCBFF51
 P 1350 7150
@@
 $EndComp
 $Comp
-L MillerLab_CommonComponents:LED_Button_connector U1
+L cage_LEDbutton_pi-rescue:LED_Button_connector-MillerLab_CommonComponents U1
 U 1 1 5DCC0482
 P 1350 5150
@@
 $EndComp
 $Comp
-L MillerLab_CommonComponents:LED_Button_connector U5
+L cage_LEDbutton_pi-rescue:LED_Button_connector-MillerLab_CommonComponents U5
 U 1 1 5DCC0AEA
 P 3150 5150
@@
 $EndComp
 $Comp
-L MillerLab_CommonComponents:LED_Button_connector U6
+L cage_LEDbutton_pi-rescue:LED_Button_connector-MillerLab_CommonComponents U6
 U 1 1 5DCC0F1E
 P 3150 5850
@@
 $EndComp
 $Comp
-L MillerLab_CommonComponents:LED_Button_connector U7
+L cage_LEDbutton_pi-rescue:LED_Button_connector-MillerLab_CommonComponents U7
 U 1 1 5DCC133F
 P 3150 6500
@@
 $EndComp
 $Comp
-L MillerLab_CommonComponents:LED_Button_connector U8
+L cage_LEDbutton_pi-rescue:LED_Button_connector-MillerLab_CommonComponents U8
 U 1 1 5DCC1766
 P 3150 7150
