File: kicad/MG_touchpad/MG_touchpad.sch (KiCad schematic (older format))
At the start: 10 parts, among them J1 Conn_01x04, Q1 BP103BF, U1 LM2904

Commit message: pcb layout for mg touchpad
Parts:
- J1: footprint (none) -> Pin_Headers:Pin_Header_Angled_1x04_Pitch2.54mm
Changed lines of the file:
@@
 EESchema Schematic File Version 4
-LIBS:MG_touchpad-cache
-EELAYER 29 0
+EELAYER 30 0
 EELAYER END
 $Descr A4 11693 8268
@@
 F 0 "J1" V 8572 2630 50  0000 L CNN
 F 1 "Conn_01x04" V 8663 2630 50  0000 L CNN
-F 2 "" H 8700 2450 50  0001 C CNN
+F 2 "Pin_Headers:Pin_Header_Angled_1x04_Pitch2.54mm" H 8700 2450 50  0001 C CNN
 F 3 "~" H 8700 2450 50  0001 C CNN
 	1    8700 2450
