File: kicad/MG_touchpad/MG_touchpad.kicad_pcb (KiCad board)
At the start: 2 copper layers, 45.2 x 13.5 mm, 10 parts, among them J1 Conn_01x04, Q1 BP103BF, U1 LM2904

Commit message: Kicad circuits -- EMG and touchpad
Parts:
- 1k: renamed from R1; value R -> 1k
- 1k: renamed from R2; value R -> 1k
- 1k: renamed from R3; value R -> 1k
- 3296Y: renamed from RV1; value R_POT -> 3296Y
- IR LED: renamed from D2; value CQY99 -> IR LED
- IR Trans: renamed from Q1; value BP103BF -> IR Transistor
- OP295: renamed from U1; value LM2904 -> OP295
- renumbered R4 to 100k, D1 to LED
Routing:
- net (no net): vias 0 -> 4
Other:
- board size 45.2 x 13.5 mm -> 45.2 x 26.7 mm
- board text added: "5V"
- board text added: "GND"
- board text added: "LED"
- board text added: "Vo"
Changed lines of the file:
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@@
   (general
     (thickness 1.6)
-    (drawings 4)
-    (tracks 69)
+    (drawings 12)
+    (tracks 73)
     (zones 0)
     (modules 10)
@@
     (solder_mask_min_width 0.25)
     (aux_axis_origin 0 0)
-    (visible_elements FFFFFF7F)
+    (visible_elements 7FFFFFFF)
     (pcbplotparams
       (layerselection 0x010fc_ffffffff)
@@
     (descr "JST PH series connector, B2B-PH-K, top entry type, through hole, Datasheet: http://www.jst-mfg.com/product/pdf/eng/ePH.pdf")
     (tags "connector jst ph")
-    (fp_text reference D1 (at 1.5 -2.8) (layer F.SilkS)
+    (fp_text reference LED (at 1.016 -2.8) (layer F.SilkS)
       (effects (font (size 1 1) (thickness 0.15)))
     )
@@
     (descr "JST PH series connector, B2B-PH-K, top entry type, through hole, Datasheet: http://www.jst-mfg.com/product/pdf/eng/ePH.pdf")
     (tags "connector jst ph")
-    (fp_text reference D2 (at 1.5 -2.8 90) (layer F.SilkS)
-      (effects (font (size 1 1) (thickness 0.15)))
-    )
-    (fp_text value CQY99 (at 1 3.8 90) (layer F.Fab)
+    (fp_text reference "IR LED" (at 1.016 -2.8 90) (layer F.SilkS)
+      (effects (font (size 1 1) (thickness 0.15)))
+    )
+    (fp_text value "IR LED" (at 1 3.8 90) (layer F.Fab)
       (effects (font (size 1 1) (thickness 0.15)))
     )
@@
     (descr "JST PH series connector, B2B-PH-K, top entry type, through hole, Datasheet: http://www.jst-mfg.com/product/pdf/eng/ePH.pdf")
     (tags "connector jst ph")
-    (fp_text reference Q1 (at 1.5 -2.8 90) (layer F.SilkS)
-      (effects (font (size 1 1) (thickness 0.15)))
-    )
-    (fp_text value BP103BF (at 1 3.8 90) (layer F.Fab)
+    (fp_text reference "IR Trans" (at 1.016 -2.8 90) (layer F.SilkS)
+      (effects (font (size 1 1) (thickness 0.15)))
+    )
+    (fp_text value "IR Transistor" (at 1 3.8 90) (layer F.Fab)
       (effects (font (size 1 1) (thickness 0.15)))
     )
@@
     (tags "resistor 1206")
     (attr smd)
-    (fp_text reference R1 (at 2.212 1.85 90) (layer B.SilkS)
-      (effects (font (size 1 1) (thickness 0.15)) (justify mirror))
-    )
-    (fp_text value R (at 0 -1.95 90) (layer B.Fab)
+    (fp_text reference 1k (at 3.122 0.254 180) (layer B.SilkS)
+      (effects (font (size 1 1) (thickness 0.15)) (justify mirror))
+    )
+    (fp_text value 1k (at 0 -1.95 90) (layer B.Fab)
       (effects (font (size 1 1) (thickness 0.15)) (justify mirror))
     )
@@
     (tags "resistor 1206")
     (attr smd)
-    (fp_text reference R2 (at 0 1.85 270) (layer B.SilkS)
-      (effects (font (size 1 1) (thickness 0.15)) (justify mirror))
-    )
-    (fp_text value R (at 0 -1.95 270) (layer B.Fab)
+    (fp_text reference 1k (at -2.868 0) (layer B.SilkS)
+      (effects (font (size 1 1) (thickness 0.15)) (justify mirror))
+    )
+    (fp_text value 1k (at 0 -1.95 270) (layer B.Fab)
       (effects (font (size 1 1) (thickness 0.15)) (justify mirror))
     )
@@
     (tags "resistor 1206")
     (attr smd)
-    (fp_text reference R3 (at 0 1.85 180) (layer B.SilkS)
-      (effects (font (size 1 1) (thickness 0.15)) (justify mirror))
-    )
-    (fp_text value R (at 0 -1.95 180) (layer B.Fab)
+    (fp_text reference 1k (at 0 1.85 180) (layer B.SilkS)
+      (effects (font (size 1 1) (thickness 0.15)) (justify mirror))
+    )
+    (fp_text value 1k (at 0 -1.95 180) (layer B.Fab)
       (effects (font (size 1 1) (thickness 0.15)) (justify mirror))
     )
@@
     (tags "resistor 1206")
     (attr smd)
-    (fp_text reference R4 (at 0 1.85 270) (layer B.SilkS)
+    (fp_text reference 100k (at 2.974 -0.254) (layer B.SilkS)
       (effects (font (size 1 1) (thickness 0.15)) (justify mirror))
     )
@@
     (descr "Spindle Trimmer Potentiometer, Bourns 3296Y, https://www.bourns.com/pdfs/3296.pdf")
     (tags "Spindle Trimmer Potentiometer   Bourns 3296Y")
-    (fp_text reference RV1 (at -9.398 3.048) (layer F.SilkS)
-      (effects (font (size 1 1) (thickness 0.15)))
-    )
-    (fp_text value R_POT (at -2.54 4.94) (layer F.Fab)
+    (fp_text reference 3296Y (at -2.54 4.572) (layer F.SilkS)
+      (effects (font (size 1 1) (thickness 0.15)))
+    )
+    (fp_text value 3296Y (at -2.54 4.94) (layer F.Fab)
       (effects (font (size 1 1) (thickness 0.15)))
     )
@@
     (descr "8-lead though-hole mounted DIP package, row spacing 7.62 mm (300 mils)")
     (tags "THT DIP DIL PDIP 2.54mm 7.62mm 300mil")
-    (fp_text reference U1 (at 3.81 -2.33) (layer F.SilkS)
-      (effects (font (size 1 1) (thickness 0.15)))
-    )
-    (fp_text value LM2904 (at 3.81 9.95) (layer F.Fab)
+    (fp_text reference OP295 (at 3.81 -2.33) (layer F.SilkS)
+      (effects (font (size 1 1) (thickness 0.15)))
+    )
+    (fp_text value OP295 (at 3.81 9.95) (layer F.Fab)
       (effects (font (size 1 1) (thickness 0.15)))
     )
@@
     (descr "Through hole angled pin header, 1x04, 2.54mm pitch, 6mm pin length, single row")
     (tags "Through hole angled pin header THT 1x04 2.54mm single row")
-    (fp_text reference J1 (at 4.385 -2.27) (layer F.SilkS)
-      (effects (font (size 1 1) (thickness 0.15)))
-    )
-    (fp_text value Conn_01x04 (at 4.385 9.89) (layer F.Fab)
+    (fp_text reference J1 (at 2.032 -2.794) (layer F.SilkS)
+      (effects (font (size 1 1) (thickness 0.15)))
+    )
+    (fp_text value Conn_01x04 (at -1.778 3.81 270) (layer F.Fab)
       (effects (font (size 1 1) (thickness 0.15)))
     )
@@
     )
   )
-  (gr_line (start 106.934 78.994) (end 106.934 65.532) (layer Edge.Cuts) (width 0.5))
-  (gr_line (start 152.146 78.994) (end 106.934 78.994) (layer Edge.Cuts) (width 0.5))
-  (gr_line (start 152.146 65.532) (end 152.146 78.994) (layer Edge.Cuts) (width 0.5))
-  (gr_line (start 106.934 65.532) (end 152.146 65.532) (layer Edge.Cuts) (width 0.5))
+  (gr_text Vo (at 108.966 68.58) (layer B.SilkS)
+    (effects (font (size 1 1) (thickness 0.15)) (justify mirror))
+  )
+  (gr_text LED (at 108.966 71.12) (layer B.SilkS)
+    (effects (font (size 1 1) (thickness 0.15)) (justify mirror))
+  )
+  (gr_text GND (at 108.966 73.66) (layer B.SilkS)
+    (effects (font (size 1 1) (thickness 0.15)) (justify mirror))
+  )
+  (gr_text 5V (at 108.966 76.454) (layer B.SilkS)
+    (effects (font (size 1 1) (thickness 0.15)) (justify mirror))
+  )
+  (gr_circle (center 146.304 63.246) (end 149.404465 63.246) (layer Margin) (width 0.127))
+  (gr_circle (center 115.316 63.246) (end 118.416465 63.246) (layer Margin) (width 0.127))
+  (gr_circle (center 115.316 81.788) (end 118.416465 81.788) (layer Margin) (width 0.127))
+  (gr_circle (center 146.304 81.788) (end 149.404465 81.788) (layer Margin) (width 0.127))
+  (gr_line (start 106.934 85.852) (end 106.934 59.182) (layer Edge.Cuts) (width 0.5))
+  (gr_line (start 152.146 85.852) (end 106.934 85.852) (layer Edge.Cuts) (width 0.5))
+  (gr_line (start 152.146 59.182) (end 152.146 85.852) (layer Edge.Cuts) (width 0.5))
+  (gr_line (start 106.934 59.182) (end 152.146 59.182) (layer Edge.Cuts) (width 0.5))
+  (via (at 115.316 63.246) (size 6.604) (drill 5.588) (layers F.Cu B.Cu) (net 0))
+  (via (at 146.304 81.788) (size 6.604) (drill 5.588) (layers F.Cu B.Cu) (net 0))
+  (via (at 115.316 81.788) (size 6.604) (drill 5.588) (layers F.Cu B.Cu) (net 0))
+  (via (at 146.304 63.246) (size 6.604) (drill 5.588) (layers F.Cu B.Cu) (net 0))
   (segment (start 135.466 76.306) (end 134.366 76.306) (width 0.25) (layer B.Cu) (net 1))
   (segment (start 136.166 77.006) (end 135.466 76.306) (width 0.25) (layer B.Cu) (net 1))
